Commit message: Changes in the frame position for the camera attachment

File: ros_stereo_vision/urdf/Stero_Setup.urdf (robot description, URDF)
Before this commit: robot stereo_robot, 2 links, 1 joints
Joints:
- joint stereo_base_camera_attachment: origin xyz=0 0 0.425 rpy=0 0 0 -> xyz=0.225 0 0.425 rpy=0 0 0

Commit message: Visualize the urdf in RVIZ and stereo camera setup is ready to detect obstacles

File: ros_stereo_vision/urdf/Stero_Setup.urdf (robot description, URDF)
Before this commit: robot stereo_robot, 2 links, 1 joints
Links:
- removed link stereo_base_link
- removed link stereo_camera_attachment
- added link stereo_base
- added link stereo_camera, mass 0.5; collision box size=0.025 0.1 0.025; visual box size=0.025 0.1 0.025
- added link stereo_horizontal_link, mass 2; collision box size=0.5 0.05 0.05; visual box size=0.5 0.05 0.05
- added link stereo_left_camera
- added link stereo_vertical_link, mass 10; collision box size=0.05 0.05 0.8; visual box size=0.05 0.05 0.8
Joints:
- added joint stereo_base_vertical: type fixed, parent stereo_base, child stereo_vertical_link, origin xyz=0.0 0.0 0.4 rpy=0 0 0
- added joint stereo_camera_camera_attachment: type fixed, parent stereo_horizontal_link, child stereo_camera, origin xyz=0.4625 0.0 -0.0375 rpy=0 -0.2617 0
- added joint stereo_left_camera_frame: type fixed, parent stereo_camera, child stereo_left_camera, origin xyz=0.0 0.035 0.0 rpy=0 1.57 0
- joint stereo_base_camera_attachment: child stereo_camera_attachment -> stereo_horizontal_link; origin xyz=0.225 0 0.425 rpy=0 0 0 -> xyz=0.0 0.0 0.425 rpy=0 0 0; parent stereo_base_link -> stereo_vertical_link

Commit message: Pose estimated from the object by using Pnp (cv2.solvePnp)

File: ros_stereo_vision/urdf/Stero_Setup.urdf (robot description, URDF)
Before this commit: robot stereo_robot, 5 links, 4 joints
Links:
- removed link stereo_horizontal_link
Joints:
- removed joint stereo_base_camera_attachment
- joint stereo_camera_camera_attachment: origin xyz=0.4625 0.0 -0.0375 rpy=0 -0.2617 0 -> xyz=0.0375 0.0 0.4 rpy=0 0 0; parent stereo_horizontal_link -> stereo_vertical_link
- joint stereo_left_camera_frame: origin xyz=0.0 0.035 0.0 rpy=0 1.57 0 -> xyz=0.0 0.035 0.0 rpy=0 0 0
